File: Automated_Aquarium/Schematic files/Automated_Aquarium_v3/Stepper_Drivers.kicad_sch (KiCad schematic)
At the start: 11 parts, among them K1 G3VM-61VY3_TR05_, K2 G3VM-61VY3_TR05_, Q2 PMOS, SW1 SW_DIP_x03

Commit message: init pcb
Parts:
- removed SW1: SW_DIP_x03, symbol Switch:SW_DIP_x03
- added S3: 218-4LPSTR, SOIC127P844X265-8N, symbol SamacSys_Parts:218-4LPSTR
- Q2: footprint (none) -> Package_TO_SOT_SMD:SOT-23; LCSC Part Number (none) -> C353080
Connections:
- net at A1.12 (MS3), R6.2: now also S3.6
- net at A1.10 (MS1), R6.2: now also S3.8
- net at A1.11 (MS2), R6.2: now also S3.7
- net at R6.1: now also S3.1, S3.2, S3.3, S3.4
Other:
- moved on the sheet: R6

Commit message: finish aqua schem, add inital layout
Parts:
- R6: LCSC Part Number C22809 -> C855633
- S3: LCSC Part Number (none) -> C2758160
Changed lines of the file:
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@@
     (stroke (width 0) (type default))
   )
-  (label "MTR1.1B" (at 151.13 82.55 0)
+  (label "MTR1.1B" (at 151.13 82.55 0) (fields_autoplaced)
     (effects (font (size 1.27 1.27)) (justify left bottom))
   )
-  (label "MTR1.2B" (at 151.13 90.17 0)
+  (label "MTR1.2B" (at 151.13 90.17 0) (fields_autoplaced)
     (effects (font (size 1.27 1.27)) (justify left bottom))
   )
-  (label "MTR1.2A" (at 151.13 87.63 0)
+  (label "MTR1.2A" (at 151.13 87.63 0) (fields_autoplaced)
     (effects (font (size 1.27 1.27)) (justify left bottom))
   )
-  (label "MTR1.1A" (at 151.13 85.09 0)
+  (label "MTR1.1A" (at 151.13 85.09 0) (fields_autoplaced)
     (effects (font (size 1.27 1.27)) (justify left bottom))
   )
@@
       (effects (font (size 1.27 1.27)) (justify left) hide)
     )
-    (property "LCSC Part Number" "C22809" (at 104.14 115.57 0)
+    (property "LCSC Part Number" "C855633" (at 104.14 115.57 0)
       (effects (font (size 1.27 1.27)) hide)
     )
@@
       (effects (font (size 1.27 1.27)) (justify left) hide)
     )
-    (property "LCSC Part Number" "C22809" (at 119.38 110.49 0)
+    (property "LCSC Part Number" "C855633" (at 119.38 110.49 0)
       (effects (font (size 1.27 1.27)) hide)
     )
@@
       (effects (font (size 1.27 1.27)) (justify left) hide)
     )
+    (property "LCSC Part Number" "C2758160" (at 73.66 92.71 0)
+      (effects (font (size 1.27 1.27)) hide)
+    )
     (pin "1")
     (pin "2")
@@
       (effects (font (size 1.27 1.27)) (justify left) hide)
     )
-    (property "LCSC Part Number" "C22809" (at 111.76 113.03 0)
+    (property "LCSC Part Number" "C855633" (at 111.76 113.03 0)
       (effects (font (size 1.27 1.27)) hide)
     )
@@
       (effects (font (size 1.27 1.27)) (justify left) hide)
     )
-    (property "LCSC Part Number" "C22809" (at 59.69 88.9 0)
-      (effects (font (size 1.27 1.27)) hide)
-    )
+    (property "LCSC Part Number" "C855633" (at 59.69 88.9 0)
+      (effects (font (size 1.27 1.27)) hide)
+    )
