File: IntegratedStepper/PCB/IntegratedStepper/Magnetic_Encoder.kicad_sch (KiCad schematic)
At the start: 0 parts

Commit message: Update Integrated Stepper PCB with ESP sch and CAN sch
Parts:
- added C16: 10uF, Capacitor_SMD:C_0603_1608Metric, symbol Device:C
- added C17: 0.1uF, Capacitor_SMD:C_0603_1608Metric, symbol Device:C
- added U2: AS5048A, Package_SO:TSSOP-14_4.4x5mm_P0.65mm, symbol Sensor_Magnetic:AS5048A
Connections:
- new net 3V3_VCC: C16.1, C17.1, U2.11 (VDD5V), U2.12 (VDD3V)
- new net GND: C16.2, C17.2, U2.13 (GND)
- new net M_CS0: U2.1 (~{CSn})
- new net M_MISO: U2.3 (MISO)
- new net M_MOSI: U2.4 (MOSI)
- new net M_PWM: U2.14 (PWM)
- new net M_SCLK: U2.2 (CLK)

Commit message: Update Integrated Stepper with inital PCB
This is going to be so hard :(
Parts:
- C17: footprint Capacitor_SMD:C_0603_1608Metric -> Capacitor_SMD:C_0603_1608Metric_Pad1.08x0.95mm_HandSolder
Changed lines of the file:
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@@
 			)
 		)
-		(property "Footprint" "Capacitor_SMD:C_0603_1608Metric"
+		(property "Footprint" "Capacitor_SMD:C_0603_1608Metric_Pad1.08x0.95mm_HandSolder"
 			(at 171.1452 83.82 0)
 			(effects

Commit message: add changes for instock parts
Parts:
- U2: LCSC (none) -> C2655181; LCSC Part (none) -> C2655181; LCSC Part Number (none) -> C2655181
Changed lines of the file:
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@@
+			)
+		)
+		(property "LCSC" "C2655181"
+			(at 143.51 93.98 0)
+			(effects
+				(font
+					(size 1.27 1.27)
+				)
+				(hide yes)
+			)
+		)
+		(property "LCSC Part" "C2655181"
+			(at 143.51 93.98 0)
+			(effects
+				(font
+					(size 1.27 1.27)
+				)
+				(hide yes)
+			)
+		)
+		(property "LCSC Part Number" "C2655181"
+			(at 143.51 93.98 0)
+			(effects
+				(font
+					(size 1.27 1.27)
+				)
+				(hide yes)
 			)
 		)

Commit message: update with more in stock parts
Parts:
- C16: LCSC (none) -> C96446; LCSC Part (none) -> C96446; LCSC Part Number (none) -> C96446
- C17: footprint Capacitor_SMD:C_0603_1608Metric_Pad1.08x0.95mm_HandSolder -> Capacitor_SMD:C_0603_1608Metric; LCSC (none) -> C2929200; LCSC Part (none) -> C2929200; LCSC Part Number (none) -> C2929200
Changed lines of the file:
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@@
 			)
 		)
-		(property "Footprint" "Capacitor_SMD:C_0603_1608Metric_Pad1.08x0.95mm_HandSolder"
+		(property "Footprint" "Capacitor_SMD:C_0603_1608Metric"
 			(at 171.1452 83.82 0)
 			(effects
@@
 		)
 		(property "Description" "Unpolarized capacitor"
+			(at 170.18 80.01 0)
+			(effects
+				(font
+					(size 1.27 1.27)
+				)
+				(hide yes)
+			)
+		)
+		(property "Voltage Rating" ""
+			(at 170.18 80.01 0)
+			(effects
+				(font
+					(size 1.27 1.27)
+				)
+				(hide yes)
+			)
+		)
+		(property "LCSC" "C2929200"
+			(at 170.18 80.01 0)
+			(effects
+				(font
+					(size 1.27 1.27)
+				)
+				(hide yes)
+			)
+		)
+		(property "LCSC Part Number" "C2929200"
+			(at 170.18 80.01 0)
+			(effects
+				(font
+					(size 1.27 1.27)
+				)
+				(hide yes)
+			)
+		)
+		(property "LCSC Part" "C2929200"
 			(at 170.18 80.01 0)
 			(effects
@@
 			(at 158.75 80.01 0)
 			(effects
+				(font
+					(size 1.27 1.27)
+				)
+				(hide yes)
+			)
+		)
+		(property "LCSC" "C96446"
+			(at 158.75 80.01 0)
+			(effects
+				(font
+					(size 1.27 1.27)
+				)
+				(hide yes)
+			)
+		)
+		(property "LCSC Part Number" "C96446"
+			(at 158.75 80.01 0)
+			(effects
+				(font
+					(size 1.27 1.27)
+				)
+				(hide yes)
+			)
+		)
+		(property "Voltage Rating" ""
+			(at 158.75 80.01 0)
+			(effects
+				(font
+					(size 1.27 1.27)
+				)
+				(hide yes)
+			)
+		)
+		(property "LCSC Part" "C96446"
+			(at 158.75 80.01 0)
+			(effects
